Commit message: Initial commit

File: assets/ASSY_Hand_R/test_fixed.urdf (robot description, URDF)
Before this commit: robot aidin_right_test, 22 links, 21 joints
Joints:
- joint joint2_baby_z: limit lower=0.1 upper=1.6707963 effort=10.0 velocity=1.5707963 -> lower=0.4 upper=1.9 effort=10.0 velocity=1.5707963
- joint joint2_index_z: limit lower=0.1 upper=1.6707963 effort=10.0 velocity=1.5707963 -> lower=0.8 upper=2.3 effort=10.0 velocity=1.5707963
- joint joint2_middle_z: limit lower=0.1 upper=1.6707963 effort=10.0 velocity=1.5707963 -> lower=0.4 upper=1.9 effort=10.0 velocity=1.5707963
- joint joint2_ring_z: limit lower=0.1 upper=1.6707963 effort=10.0 velocity=1.5707963 -> lower=0.4 upper=1.9 effort=10.0 velocity=1.5707963
- joint joint2_thumb_z: limit lower=0.0 upper=1.1 effort=10.0 velocity=1.5707963 -> lower=0.01 upper=1.6 effort=10.0 velocity=1.5707963
- joint joint3_baby_z: limit lower=0.1 upper=1.634464 effort=10.0 velocity=1.5707963 -> lower=0.05 upper=1.55 effort=10.0 velocity=1.5707963
- joint joint3_index_z: limit lower=0.0 upper=1.634464 effort=10.0 velocity=1.5707963 -> lower=0.05 upper=1.55 effort=10.0 velocity=1.5707963
- joint joint3_middle_z: limit lower=0.0 upper=1.634464 effort=10.0 velocity=1.5707963 -> lower=0.05 upper=1.55 effort=10.0 velocity=1.5707963
- joint joint3_ring_z: limit lower=0.0 upper=1.634464 effort=10.0 velocity=1.5707963 -> lower=0.05 upper=1.55 effort=10.0 velocity=1.5707963
- joint joint3_thumb_z: limit lower=0.0 upper=1.1 effort=10.0 velocity=1.5707963 -> lower=0.01 upper=1.6 effort=10.0 velocity=1.5707963
- joint joint4_baby_z: limit lower=0.1 upper=1.6089969 effort=0 velocity=0 -> lower=0.05 upper=1.55 effort=0 velocity=0
- joint joint4_index_z: limit lower=0.0 upper=1.6089969 effort=0 velocity=0 -> lower=0.05 upper=1.55 effort=0 velocity=0
- joint joint4_middle_z: limit lower=0.0 upper=1.6089969 effort=0 velocity=0 -> lower=0.05 upper=1.55 effort=0 velocity=0
- joint joint4_ring_z: limit lower=0.0 upper=1.6089969 effort=0 velocity=0 -> lower=0.05 upper=1.55 effort=0 velocity=0
- joint joint4_thumb_z: mimic joint=joint3_thumb_z multiplier=-1.1 offset=0.0 -> joint=joint3_thumb_z multiplier=1.1 offset=0.0

Commit message: Collision Loss etc

File: assets/ASSY_Hand_R/test_fixed.urdf (robot description, URDF)
Before this commit: robot aidin_right_test, 22 links, 21 joints
Joints:
- joint joint2_index_z: limit lower=0.8 upper=2.3 effort=10.0 velocity=1.5707963 -> lower=0.0 upper=1.5708 effort=10.0 velocity=1.5707963; origin xyz=0 0 0.01035 rpy=-1.5708 0 1.5708 -> xyz=0 0 0.01035 rpy=-1.5708 -0.78 1.5708
- joint joint2_middle_z: limit lower=0.4 upper=1.9 effort=10.0 velocity=1.5707963 -> lower=0.3 upper=1.8708 effort=10.0 velocity=1.5707963
- joint joint2_thumb_z: limit lower=0.01 upper=1.6 effort=10.0 velocity=1.5707963 -> lower=0.01 upper=1.57 effort=10.0 velocity=1.5707963
- joint joint3_thumb_z: limit lower=0.01 upper=1.6 effort=10.0 velocity=1.5707963 -> lower=0.01 upper=1.57 effort=10.0 velocity=1.5707963
- joint joint4_baby_z: mimic joint=joint3_baby_z multiplier=1.1 offset=0.0 -> joint=joint3_baby_z multiplier=1.0 offset=0.0
- joint joint4_index_z: mimic joint=joint3_index_z multiplier=1.1 offset=0.0 -> joint=joint3_index_z multiplier=1.0 offset=0.0
- joint joint4_middle_z: mimic joint=joint3_middle_z multiplier=1.1 offset=0.0 -> joint=joint3_middle_z multiplier=1.0 offset=0.0
- joint joint4_ring_z: mimic joint=joint3_ring_z multiplier=1.1 offset=0.0 -> joint=joint3_ring_z multiplier=1.0 offset=0.0
- joint joint4_thumb_z: limit lower=0.1 upper=1.6 effort=0 velocity=0 -> lower=0.01 upper=1.57 effort=0 velocity=0; mimic joint=joint3_thumb_z multiplier=1.1 offset=0.0 -> joint=joint3_thumb_z multiplier=1.0 offset=0.0
